File: hw/hw2/hw2breakout/hw2breakout.kicad_pcb (KiCad board)
At the start: 2 copper layers, 41.9 x 23.5 mm, 8 parts, among them J1 Conn_01x03_Pin, J2 Conn_01x03_Pin, J3 Conn_01x03_Pin, U1 PCT2075DP

Commit message: rev 2 for hw2
Parts:
- removed J2, J3: Conn_01x03_Pin, Connector_PinHeader_2.54mm:PinHeader_1x03_P2.54mm_Vertical
- added C1: 0.1uF, Capacitor_THT:C_Disc_D5.0mm_W2.5mm_P2.50mm, F.Cu at (137.2, 54.8)
- added R3: 1.5k, Resistor_THT:R_Axial_DIN0207_L6.3mm_D2.5mm_P10.16mm_Horizontal, F.Cu at (125.1, 61.0)
- added R4: 1.5k, Resistor_THT:R_Axial_DIN0207_L6.3mm_D2.5mm_P10.16mm_Horizontal, F.Cu at (125.1, 66.0)
- added R5: 1.5k, Resistor_THT:R_Axial_DIN0207_L6.3mm_D2.5mm_P10.16mm_Horizontal, F.Cu at (125.0, 70.6)
- D1: footprint LED_SMD:LED_0805_2012Metric -> LED_SMD:LED_0805_2012Metric_Pad1.15x1.40mm_HandSolder
- J1: value Conn_01x03_Pin -> Conn_01x10_Pin; footprint Connector_PinHeader_2.54mm:PinHeader_1x03_P2.54mm_Vertical -> Connector_PinHeader_2.54mm:PinHeader_1x10_P2.54mm_Vertical
- TH1: footprint Resistor_SMD:R_0603_1608Metric -> Resistor_SMD:R_0603_1608Metric_Pad0.98x0.95mm_HandSolder
- moved D1 55.8 mm to (111.8, 45.1), turned to 0 degrees
- moved R1 42.8 mm to (126.0, 49.8), turned to 180 degrees
- moved TH1 40.0 mm to (124.7, 55.9), turned to 180 degrees
- moved R2 37.9 mm to (126.0, 45.1), turned to 180 degrees
- moved U1 34.1 mm to (117.3, 54.9), turned to -90 degrees
- moved J1 32.4 mm to (129.5, 49.2)
Connections:
- J1 pad 1: Net-(J1-Pin_1) -> LED_Vin
- J1 pad 2: Net-(J1-Pin_2) -> VCC
- J1 pad 3: Net-(J1-Pin_3) -> GND
- R1 pad 1: Net-(J3-Pin_2) -> Th_Out
- R2 pad 1: VCC -> LED_Vin
- TH1 pad 2: Net-(J3-Pin_2) -> Th_Out
- U1 pad 1: Net-(J2-Pin_3) -> SDA
- U1 pad 2: Net-(J2-Pin_2) -> SCL
- U1 pad 3: Net-(J2-Pin_1) -> OS
- U1 pad 5: Net-(J1-Pin_3) -> A2
- U1 pad 6: Net-(J1-Pin_2) -> A1
- U1 pad 7: Net-(J1-Pin_1) -> A0
Routing:
- net OS: track 0.00 -> 47.2 mm
- net SCL: track 0.00 -> 44.8 mm
- net A0: track 0.00 -> 38.8 mm
- net A1: track 0.00 -> 38.7 mm
- net A2: track 0.00 -> 38.1 mm
- net VCC: track 47.9 -> 80.7 mm
- net SDA: track 0.00 -> 28.7 mm
- net Th_Out: track 0.00 -> 13.1 mm
- net Net-(J3-Pin_2): track 11.2 -> 0.00 mm
- net GND: track 41.5 -> 49.8 mm
- net LED_Vin: track 0.00 -> 7.02 mm
- net Net-(J1-Pin_3): track 6.64 -> 0.00 mm
- net Net-(J2-Pin_1): track 6.20 -> 0.00 mm
- net Net-(J1-Pin_2): track 6.05 -> 0.00 mm
- net Net-(J1-Pin_1): track 5.86 -> 0.00 mm
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Other:
- board size 41.9 x 23.5 mm -> 30.5 x 33 mm
- board text added: "LED_Vin"
- board text added: "Th_Out"
- board text removed: "THOut"

Commit message: minor revisions for hw2
Routing:
- net GND: track 49.8 -> 46.0 mm
Changed lines of the file:
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@@
     (property "ki_keywords" "capacitor cap")
     (attr through_hole)
-    (fp_text reference "C1" (at 1.25 -2.5 90) (layer "F.SilkS")
+    (fp_text reference "C1" (at -2.961 0.635 90) (layer "F.SilkS")
         (effects (font (size 1 1) (thickness 0.15)))
     )
@@
   (segment (start 137.16 52.324) (end 131.628 52.324) (width 0.25) (layer "F.Cu") (net 1))
   (segment (start 131.628 52.324) (end 131.572 52.268) (width 0.25) (layer "F.Cu") (net 1))
-  (segment (start 116.373 50.333) (end 115.824 49.784) (width 0.25) (layer "F.Cu") (net 1))
   (segment (start 110.744 45.085) (end 110.744 43.18) (width 0.25) (layer "F.Cu") (net 1))
   (segment (start 129.032 42.672) (end 131.572 45.212) (width 0.25) (layer "F.Cu") (net 1))
-  (segment (start 115.316 49.657) (end 115.316 50.292) (width 0.25) (layer "F.Cu") (net 1))
   (segment (start 110.744 45.085) (end 115.316 49.657) (width 0.25) (layer "F.Cu") (net 1))
-  (segment (start 116.373 52.714) (end 116.373 50.333) (width 0.25) (layer "F.Cu") (net 1))
   (segment (start 131.572 45.212) (end 131.572 52.268) (width 0.25) (layer "F.Cu") (net 1))
   (segment (start 111.252 42.672) (end 129.032 42.672) (width 0.25) (layer "F.Cu") (net 1))

Commit message: minor rev
Parts:
- J1: moved to B.Cu
- moved C1 0.63 mm to (136.5, 54.8)
- turned J1 to 180 degrees
Routing:
- net GND: track 46.0 -> 40.4 mm
Other:
- board text added: "remy"
- board text added: "swag money :D"
