File: EE193ConceptualDesign/Team Temp Sensor.kicad_pcb (KiCad board)
At the start: 2 copper layers, 27.4 x 62.2 mm, 35 parts, among them J1 USB_B_Micro, J2 Battery_Connector, Q1 BC818, Q2 BC818, SW1 SW_DPDT_x2, SW2 SW_DIP_x01, U1 ESP32-C3-WROOM-02, U2 CP2102N-A02-GQFN28, U3 LD1117S33TR_SOT223

Commit message: v0.3 schematic, layout WIP
Parts:
- removed C1, C10, C4, C8: 10 uF, Capacitor_SMD:C_0805_2012Metric_Pad1.18x1.45mm_HandSolder
- removed C11, C2, C9: 0.1 uF, Capacitor_SMD:C_0805_2012Metric_Pad1.18x1.45mm_HandSolder
- removed C3, C5: 1 uF, Capacitor_SMD:C_0805_2012Metric_Pad1.18x1.45mm_HandSolder
- removed C6, C7: 22 pF, Capacitor_SMD:C_0805_2012Metric_Pad1.18x1.45mm_HandSolder
- removed D1: MBR0540, Diode_SMD:D_SOD-123
- removed D2, D3, D4: 1N914WT, Diode_SMD:D_SOD-523
- removed J1: USB_B_Micro, Connector_USB:USB_Micro-B_GCT_USB3076-30-A
- removed J2: Battery_Connector, Connector_JST:JST_PH_S2B-PH-K_1x02_P2.00mm_Horizontal
- removed Q1, Q2: BC818, Package_TO_SOT_SMD:SOT-23
- removed R1, R2, R5, R6, R7: 10k, Resistor_SMD:R_0805_2012Metric_Pad1.20x1.40mm_HandSolder
- removed R10, R11, R8, R9: 0, Resistor_SMD:R_0805_2012Metric_Pad1.20x1.40mm_HandSolder
- removed R3: 47.5k, Resistor_SMD:R_0805_2012Metric_Pad1.20x1.40mm_HandSolder
- removed R4: 1k, Resistor_SMD:R_0805_2012Metric_Pad1.20x1.40mm_HandSolder
- removed SW1: SW_DPDT_x2, Connector_PinHeader_2.54mm:PinHeader_1x03_P2.54mm_Vertical
- removed SW2: SW_DIP_x01, Connector_PinHeader_2.54mm:PinHeader_1x02_P2.54mm_Vertical
- removed U1: ESP32-C3-WROOM-02, espressif kicad-libraries main footprints-Espressif:ESP32-C3-WROOM-02
- removed U2: CP2102N-A02-GQFN28, CP2102N_A02_GQFN28:QFN50P500X500X80-29N
- removed U3: LD1117S33TR_SOT223, Package_TO_SOT_SMD:SOT-223-3_TabPin2
Routing:
- net Net-(D1-A): track 113.3 -> 0.00 mm
- net GND: track 96.6 -> 0.00 mm, vias 18 -> 0
- net Net-(U2-VDD): track 85.2 -> 0.00 mm, vias 2 -> 0
- net +3V3: track 70.8 -> 0.00 mm, vias 1 -> 0
- net Net-(J2-Pin_2): track 59.0 -> 0.00 mm
- net Net-(Q1-C): track 57.9 -> 0.00 mm, vias 3 -> 0
- net PowerToESP32: track 45.3 -> 0.00 mm
- net Net-(U2-GPIO.0/TXT): track 40.3 -> 0.00 mm
- net Net-(Q2-C): track 39.0 -> 0.00 mm, vias 2 -> 0
- net Net-(D3-A): track 38.9 -> 0.00 mm
- net Net-(U2-~{RST}): track 37.4 -> 0.00 mm
- net Net-(D4-A): track 34.7 -> 0.00 mm, vias 2 -> 0
- net Net-(U2-~{SUSPEND}): track 34.4 -> 0.00 mm
- net +5V: track 34.1 -> 0.00 mm
- net Net-(U1-GPIO8): track 29.0 -> 0.00 mm, vias 2 -> 0
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- removed copper zone on B.Cu, net GND
Other:
- board outline removed
- board text removed: "Board By: Alex, Amitav, and Remy Board Revision: v0.2"
- board text removed: "C10|10 uF"
- board text removed: "C11|0.1 uF"
- board text removed: "C1|10 uF"
- board text removed: "C2|0.1 uF"
- board text removed: "C3 | 1 uF"
- board text removed: "C4|10 uF"
- board text removed: "C5|10 uF"
- board text removed: "C6|22 pF"
- board text removed: "C7|22 pF"
- board text removed: "C8|10 uF"
- board text removed: "C9|0.1 uF"
- board text removed: "G"
- board text removed: "SW1|ESP32 Power"
- board text removed: "SW2|UART Power"
- board text removed: "Tufts EE193: Network Embedded Sys. Prof. Bell - Don't Move Me!"
- board text removed: "||+3V3"
- board text removed: "||Battery"
- board text removed: "||To ESP32"
