File: EE193ConceptualDesign/Team Temp Sensor.kicad_sch (KiCad schematic)
At the start: 33 parts, among them J1 USB_B_Micro, Q1 BC818, Q2 BC818, SW1 SW_DIP_x01, U1 ESP32-C3-WROOM-02, U2 CP2102N-A02-GQFN28, U3 LD1117S33TR_SOT223

Commit message: new layout revision
Parts:
- removed SW1: SW_DIP_x01, Connector_PinHeader_2.54mm:PinHeader_1x02_P2.54mm_Vertical, symbol Switch:SW_DIP_x01
- added J2: Battery_Connector, Connector_JST:JST_PH_S2B-PH-K_1x02_P2.00mm_Horizontal, symbol Connector:Conn_01x02_Pin
- added SW1: SW_DPDT_x2, Connector_PinHeader_2.54mm:PinHeader_1x03_P2.54mm_Vertical, symbol Switch:SW_DPDT_x2
- added SW2: SW_DIP_x01, Connector_PinHeader_2.54mm:PinHeader_1x02_P2.54mm_Vertical, symbol Switch:SW_DIP_x01
- C1, C10, C11, C2, C3, C4, C5, C6, C7, C8, C9: footprint Capacitor_THT:C_Disc_D8.0mm_W2.5mm_P5.00mm -> Capacitor_SMD:C_0805_2012Metric_Pad1.18x1.45mm_HandSolder
- R1, R10, R11, R2, R3, R4, R5, R6, R7, R8, R9: footprint Resistor_THT:R_Axial_DIN0207_L6.3mm_D2.5mm_P10.16mm_Horizontal -> Resistor_SMD:R_0805_2012Metric_Pad1.20x1.40mm_HandSolder
Connections:
- net +3V3: now also SW1.1 (A), SW2.2; no longer C1.2, C2.2, R1.1, U1.1 (3V3)
- net GND: now also J2.1 (Pin_1)
- net at C4.1, R4.1, U2.6 (VDD)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: now also SW2.1
- net SDA: now reaches U1.5 (GPIO6)
- net SCL: now reaches U1.6 (GPIO7)
- new net: J2.2 (Pin_2), SW1.3 (C)
- new net PowerToESP32: C1.2, C2.2, R1.1, SW1.2 (B), U1.1 (3V3)
- no-connect marks 30 -> 28

Commit message: schematic changes
Parts:
- removed SW1: SW_DPDT_x2, Connector_PinHeader_2.54mm:PinHeader_1x03_P2.54mm_Vertical, symbol Switch:SW_DPDT_x2
- added Q3: BS170F, Package_TO_SOT_SMD:SOT-23, symbol Transistor_FET:BS170F
- added U4: MCP9808_MSOP, Package_SO:MSOP-8_3x3mm_P0.65mm, symbol Sensor_Temperature:MCP9808_MSOP
Connections:
- net PowerToESP32 is gone; now on net +3V3: C1.2, C2.2, R1.1, U1.1 (3V3)
- net +3V3: now also Q3.3 (D)
- net +5V: no longer C8.1, C9.1, U3.3 (VI)
- net GND: now also U4.4 (GND), U4.5 (A2), U4.6 (A1), U4.7 (A0)
- net SCL: now also U1.15 (GPIO3/ADC1_CH3), U4.2 (SCL); no longer U1.6 (GPIO7)
- net SDA: now also U1.16 (GPIO2/ADC1_CH2), U4.1 (SDA); no longer U1.5 (GPIO6)
- net VBatt: now reaches J2.2 (Pin_2)
- net TempIC_Power: now reaches U1.3 (GPIO4/ADC1_CH4)
- net TempIC_Power: now also Q3.1 (G)
- new net: Q3.2 (S), U4.8 (V_{DD})
- new net VReg_In: C8.1, C9.1, U3.3 (VI)

Commit message: v0.3 schematic, layout WIP
Parts:
- added D5: BAS_52-02V_H6327, SODFL1608X59N, symbol BAS_52-02V_H6327:BAS_52-02V_H6327
- added Q4: NTA4151PT1G, Package_TO_SOT_SMD:SOT-416, symbol NTA4151PT1G:NTA4151PT1G
- added R12: 5.1k, Resistor_SMD:R_0805_2012Metric_Pad1.20x1.40mm_HandSolder, symbol Device:R
Connections:
- net +5V: now also D5.2 (A), Q4.1 (G), R12.2
- net GND: now also R12.1
- net VBatt: now also Q4.3 (D)
- net VReg_In: now also D5.1 (K), Q4.2 (S)
Other:
- note added: "1-Gate 2-Source 3-Drain"
- moved on the sheet: J2, Q3, U4
