File: EE193PreliminaryDesign/TeamTempSensorEE31/TeamTempSensorEE31_v0_4.kicad_pcb (KiCad board)
At the start: 2 copper layers, 27.4 x 33.7 mm, 39 parts, among them J1 USB_B_Micro, J2 Battery_Connector, Q1 BS170F, Q2 BC818, Q3 BC818, Q4 NTA4151PT1G, SW1 SW_DIP_x01, U1 CP2102N-A02-GQFN28, U2 MCP9808_MSOP, U3 LD1117S33TR_SOT223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

Commit message: v0.4 complete layout
Other:
- board text added: "Board By: Alex, Amitav, and Remy Board Revision: v0.2"
- board text removed: "Board By: Alex, Amitav, and Remy Board Revision: v0.4"
Changed lines of the file:
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@@
     )
   )
-  (gr_text "Board By: Alex, Amitav, and Remy\nBoard Revision: v0.4" (at 171.069 89.916) (layer "F.SilkS")
+  (gr_text "Board By: Alex, Amitav, and Remy\nBoard Revision: v0.2" (at 171.069 89.916) (layer "F.SilkS")
     (effects (font (face "HelveticaNeue MediumCond") (size 1 1) (thickness 0.15)) (justify left bottom))
-    (render_cache "Board By: Alex, Amitav, and Remy\nBoard Revision: v0.4" 0
+    (render_cache "Board By: Alex, Amitav, and Remy\nBoard Revision: v0.2" 0
       (polygon
         (pts
@@
       (polygon
         (pts
-          (xy 181.849146 89.399907)          (xy 181.957101 89.399907)          (xy 181.957101 89.527158)          (xy 181.849146 89.527158)
-          (xy 181.849146 89.746)          (xy 181.69796 89.746)          (xy 181.69796 89.527158)          (xy 181.343808 89.527158)
-          (xy 181.343808 89.399907)          (xy 181.472524 89.399907)          (xy 181.69796 89.399907)          (xy 181.69796 88.992755)
-          (xy 181.695273 88.992755)          (xy 181.472524 89.399907)          (xy 181.343808 89.399907)          (xy 181.343808 89.390138)
-          (xy 181.686725 88.761212)          (xy 181.849146 88.761212)
-        )
-      )
+          (xy 181.940249 89.611666)          (xy 181.538469 89.611666)          (xy 181.54625 89.589784)          (xy 181.555372 89.569091)
+          (xy 181.565731 89.549491)          (xy 181.577223 89.530888)          (xy 181.589744 89.513185)          (xy 181.60319 89.496287)
+          (xy 181.617455 89.480098)          (xy 181.632438 89.464521)          (xy 181.648032 89.44946)          (xy 181.664135 89.43482)
+          (xy 181.680641 89.420503)          (xy 181.697447 89.406415)          (xy 181.714448 89.392458)          (xy 181.731541 89.378537)
+          (xy 181.748621 89.364556)          (xy 181.765584 89.350418)          (xy 181.782326 89.336027)          (xy 181.798743 89.321288)
+          (xy 181.814731 89.306104)          (xy 181.830184 89.290379)          (xy 181.845 89.274017)          (xy 181.859074 89.256922)
+          (xy 181.872302 89.238998)          (xy 181.88458 89.220148)          (xy 181.895804 89.200277)          (xy 181.905869 89.179289)
+          (xy 181.914671 89.157086)          (xy 181.922106 89.133574)          (xy 181.928071 89.108656)          (xy 181.93246 89.082236)
+          (xy 181.93517 89.054218)          (xy 181.936096 89.024506)          (xy 181.935869 89.01118)          (xy 181.93518 88.998003)
+          (xy 181.934021 88.984994)          (xy 181.932384 88.97217)          (xy 181.930258 88.95955)          (xy 181.927636 88.94715)
+          (xy 181.924508 88.934991)          (xy 181.920866 88.923088)          (xy 181.9167 88.911461)          (xy 181.912002 88.900126)
+          (xy 181.906762 88.889103)          (xy 181.900973 88.878408)          (xy 181.894624 88.868061)          (xy 181.887708 88.858078)
+          (xy 181.880214 88.848478)          (xy 181.872135 88.839278)          (xy 181.863462 88.830498)          (xy 181.854185 88.822153)
+          (xy 181.844295 88.814264)          (xy 181.833784 88.806846)          (xy 181.822643 88.799919)          (xy 181.810863 88.7935)
+          (xy 181.798434 88.787608)          (xy 181.785349 88.782259)          (xy 181.771598 88.777473)          (xy 181.757172 88.773266)
+          (xy 181.742063 88.769658)          (xy 181.726261 88.766665)          (xy 181.709758 88.764307)          (xy 181.692544 88.7626)
+          (xy 181.674611 88.761562)          (xy 181.65595 88.761212)          (xy 181.636523 88.761568)          (xy 181.617848 88.762629)
+          (xy 181.599916 88.764386)          (xy 181.58272 88.766831)          (xy 181.566249 88.769955)          (xy 181.550494 88.773749)
+          (xy 181.535448 88.778205)          (xy 181.521101 88.783313)          (xy 181.507444 88.789064)          (xy 181.494469 88.79545)
+          (xy 181.482165 88.802462)          (xy 181.470525 88.810092)          (xy 181.45954 88.81833)          (xy 181.4492 88.827167)
+          (xy 181.439497 88.836596)          (xy 181.430422 88.846606)          (xy 181.421966 88.857189)          (xy 181.41412 88.868337)
+          (xy 181.406875 88.88004)          (xy 181.400222 88.89229)          (xy 181.394153 88.905078)          (xy 181.388658 88.918395)
+          (xy 181.383729 88.932232)          (xy 181.379356 88.946581)          (xy 181.375532 88.961433)          (xy 181.372245 88.976778)
+          (xy 181.369489 88.992608)          (xy 181.367254 89.008915)          (xy 181.365532 89.025689)          (xy 181.364312 89.042922)
+          (xy 181.363587 89.060604)          (xy 181.363347 89.078728)          (xy 181.514533 89.078728)          (xy 181.514782 89.059959)
+          (xy 181.515606 89.041221)          (xy 181.517122 89.022677)          (xy 181.519449 89.00449)          (xy 181.522703 88.986822)
+          (xy 181.527001 88.969836)          (xy 181.532462 88.953696)          (xy 181.539202 88.938563)          (xy 181.547339 88.924601)
+          (xy 181.55699 88.911973)          (xy 181.568272 88.90084)          (xy 181.581303 88.891367)          (xy 181.596201 88.883716)
+          (xy 181.613082 88.878049)          (xy 181.632063 88.874529)          (xy 181.642379 88.873626)          (xy 181.653263 88.87332)
+          (xy 181.669176 88.874102)          (xy 181.683868 88.876395)          (xy 181.697365 88.880117)          (xy 181.709695 88.885188)
+          (xy 181.720884 88.891528)          (xy 181.73096 88.899054)          (xy 181.739948 88.907687)          (xy 181.747877 88.917345)
+          (xy 181.754772 88.927947)          (xy 181.760661 88.939413)          (xy 181.76557 88.951662)          (xy 181.769527 88.964613)
+          (xy 181.772557 88.978185)          (xy 181.774689 88.992298)          (xy 181.775948 89.006869)          (xy 181.776362 89.021819)
+          (xy 181.775169 89.049542)          (xy 181.771693 89.075556)          (xy 181.766086 89.099999)          (xy 181.7585 89.123011)
+          (xy 181.749086 89.144728)          (xy 181.737999 89.165289)          (xy 181.725389 89.184832)          (xy 181.711408 89.203494)
+          (xy 181.69621 89.221414)          (xy 181.679947 89.23873)          (xy 181.662769 89.255579)          (xy 181.644831 89.272099)
+          (xy 181.626284 89.288429)          (xy 181.60728 89.304707)          (xy 181.587972 89.32107)          (xy 181.568511 89.337656)
+          (xy 181.54905 89.354604)          (xy 181.529742 89.372051)          (xy 181.510738 89.390135)          (xy 181.492191 89.408994)
+          (xy 181.474253 89.428767)          (xy 181.457075 89.449591)          (xy 181.440812 89.471604)          (xy 181.425614 89.494945)
+          (xy 181.411633 89.51975)          (xy 181.399023 89.546158)          (xy 181.387936 89.574308)          (xy 181.378523 89.604336)
+          (xy 181.370936 89.636382)          (xy 181.365329 89.670582)          (xy 181.361853 89.707075)          (xy 181.36066 89.746)
+          (xy 181.940249 89.746)
+        )
+      )

Commit message: change font on v0.4
Other:
- board text added: "Team: Alex, Amitav, and Remy Board Revision: v0.2"
- board text added: "Tufts EE193 Net. Embed. Sys. Prof. Bell - Don't Move Me!"
- board text removed: "Board By: Alex, Amitav, and Remy Board Revision: v0.2"
- board text removed: "Tufts EE193: Net. Embedded Sys. Prof. Bell - Don't Move Me!"
